Commit message: Replaced rtbmap with Mola LIO

File: robot/src/workspace/src/kapibara/description/robot_core.xacro (robot description, xacro)
@@ -171,5 +171,5 @@
     </gazebo>
     <!-- RIGHT WHEEL LINK -->
-    <joint name="$(arg robot_name)_wheel_right1_joint" type="continuous">
+    <joint name="$(arg robot_name)_wheel_right2_joint" type="continuous">
         <mimic joint="$(arg robot_name)_wheel_right3_joint" multiplier="1" offset="0"/>
         <parent link="$(arg robot_name)_chassis" />
@@ -203,5 +203,5 @@
         <mu2 value="0.5"/>
     </gazebo>
-    <joint name="$(arg robot_name)_wheel_right2_joint" type="continuous">
+    <joint name="$(arg robot_name)_wheel_right1_joint" type="continuous">
         <mimic joint="$(arg robot_name)_wheel_right3_joint" multiplier="1" offset="0"/>
         <parent link="$(arg robot_name)_chassis" />
